File: CBS logic with variable blend.kicad_pcb (KiCad board)
At the start: 2 copper layers, 98.8 x 100 mm, 115 parts, among them J1 AC_IN, Q1 MPSA18, Q10 MPSA55, Q2 MPSA18, Q3 MPSA18, Q4 MPSA18, Q5 2N5461, Q7 MPSA55, Q8 MPSA55, Q9 MPSA18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

Commit message: Minor corrections.
Parts:
- moved C40 2.12 mm to (109.2, 115.3), turned to 180 degrees
- moved C41 2.12 mm to (109.2, 120.4), turned to 180 degrees
- moved C43 0.38 mm to (109.2, 128.1)
- moved C42 0.28 mm to (109.2, 133.2)
Connections:
- C40 pad 1: Left_Front_OUT -> Net-(C40-Pad1)
- C40 pad 2: Net-(C40-Pad2) -> Left_Front_OUT
- C41 pad 1: Right_Front_OUT -> Net-(C41-Pad1)
- C41 pad 2: Net-(C41-Pad2) -> Right_Front_OUT
- U3 pad 2: Net-(C41-Pad2) -> Net-(C41-Pad1)
- U3 pad 6: Net-(C40-Pad2) -> Net-(C40-Pad1)
Routing:
- net Net-(C41-Pad2): track 14.0 -> 0.00 mm
- net Net-(C41-Pad1): track 0.00 -> 14.0 mm
- net Net-(C40-Pad2): track 8.77 -> 0.00 mm
- net Net-(C40-Pad1): track 0.00 -> 8.77 mm
