File: CBS logic with variable blend.sch (KiCad schematic (older format))
At the start: 115 parts, among them J1 AC_IN, Q1 MPSA18, Q10 MPSA55, Q2 MPSA18, Q3 MPSA18, Q4 MPSA18, Q5 2N5461, Q7 MPSA55, Q8 MPSA55, Q9 MPSA18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

Commit message: Minor corrections.
Parts:
- C40, C41, C42, C43: symbol Device:C -> Device:CP
- C6: value 180n -> 18n
Connections:
- net Left_Front_OUT: now also C40.2; no longer C40.1
- net Right_Front_OUT: now also C41.2; no longer C41.1
- net at U3.2: now also C41.1; no longer C41.2
- net at U3.6: now also C40.1; no longer C40.2
Changed lines of the file:
@@
 P 1800 4300
 F 0 "C6" H 1915 4346 50  0000 L CNN
-F 1 "180n" H 1850 4150 50  0000 L CNN
+F 1 "18n" H 1850 4150 50  0000 L CNN
 F 2 "Capacitor_THT:C_Disc_D5.0mm_W2.5mm_P2.50mm" H 1838 4150 50  0001 C CNN
 F 3 "~" H 1800 4300 50  0001 C CNN
@@
 	5750 5400 4950 5400
 $Comp
-L Device:C C41
+L Device:CP C41
 U 1 1 5ED39C79
 P 6700 5000
@@
 F 3 "~" H 6700 5000 50  0001 C CNN
 	1    6700 5000
-	1    0    0    -1
-$EndComp
-Wire Wire Line
-	6700 5400 6700 5150
+	1    0    0    1
+$EndComp
 Text GLabel 6800 4800 2    50   UnSpc ~ 0
 Right_Front_OUT
-Wire Wire Line
-	6700 4850 6700 4800
-Wire Wire Line
-	6700 4800 6800 4800
-$Comp
-L Device:C C40
+$Comp
+L Device:CP C40
 U 1 1 5ED89E67
 P 6400 4850
@@
 F 3 "~" H 6400 4850 50  0001 C CNN
 	1    6400 4850
-	1    0    0    -1
-$EndComp
-Wire Wire Line
-	6300 5400 6300 5050
-Wire Wire Line
-	6300 5050 6400 5050
-Wire Wire Line
-	6400 5050 6400 5000
-Wire Wire Line
-	6400 4700 6450 4700
-Wire Wire Line
-	6450 4700 6450 4600
-Wire Wire Line
-	6450 4600 6400 4600
+	1    0    0    1
+$EndComp
 Text GLabel 6400 4600 0    50   UnSpc ~ 0
 Left_Front_OUT
 $Comp
-L Device:C C42
+L Device:CP C42
 U 1 1 5EE78A22
 P 6650 6550
@@
 	6650 6800 6650 6700
 $Comp
-L Device:C C43
+L Device:CP C43
 U 1 1 5EEDCAFD
 P 5850 7050
@@
 Wire Wire Line
 	650  2850 850  2850
+Wire Wire Line
+	6700 5400 6700 5150
+Wire Wire Line
+	6700 4850 6700 4800
+Wire Wire Line
+	6700 4800 6800 4800
+Wire Wire Line
+	6400 5000 6300 5000
+Wire Wire Line
+	6300 5000 6300 5400
+Wire Wire Line
+	6400 4700 6400 4600
 $EndSCHEMATC
